File: pcb/vdp_cartridge_20k_3rd/vdp_cartridge.kicad_pcb (KiCad board)
At the start: 2 copper layers, 95.2 x 65.4 mm, 26 parts, among them J1 Conn_01x06_Pin, Q1 NMOS, Q2 NMOS, Q3 NMOS

Commit message: *
Parts:
- removed C7, C9: 0.1uF, Capacitor_SMD:C_0402_1005Metric
- removed U1: ~, My Parts:CLOCK
- removed U5, U6: ~, Package_SO:SSOP-24_5.3x8.2mm_P0.65mm
- added U7: 74LVC541, Package_SO:TSSOP-20_4.4x6.5mm_P0.65mm, F.Cu at (126.1, 88.2)
- added U8: 74LVC541, Package_SO:TSSOP-20_4.4x6.5mm_P0.65mm, F.Cu at (137.8, 88.2)
- added X1: SG-8002DC, Package_DIP:DIP-8_W7.62mm, F.Cu at (96.6, 40.1)
- C2, C4, C5, C6, C8: footprint Capacitor_SMD:C_0402_1005Metric -> Capacitor_SMD:C_0603_1608Metric_Pad1.08x0.95mm_HandSolder
- Q1, Q2, Q3: value NMOS -> BSS138; footprint 0-My_Parts:MOSFET(SMD) -> Package_TO_SOT_SMD:SOT-23
- U4: footprint Package_SO:SSOP-24_5.3x8.2mm_P0.65mm -> Package_SO:TSSOP-24_4.4x5mm_P0.4mm
Connections:
- Q1 pad 1: /BUSDIR -> SLOT_DATA_DIR
- Q1 pad 2: SLOT_DATA_DIR -> GND
- Q1 pad 3: GND -> /BUSDIR
- Q2 pad 1: /WAIT -> SLOT_WAIT
- Q2 pad 2: SLOT_WAIT -> GND
- Q2 pad 3: GND -> /WAIT
- Q3 pad 1: /INT -> SLOT_INT
- Q3 pad 2: SLOT_INT -> GND
- Q3 pad 3: GND -> /INT
