File: pcb/vdp_cartridge_20k_3rd/vdp_cartridge.kicad_sch (KiCad schematic)
At the start: 24 parts, among them J1 Conn_01x06_Pin, Q1 NMOS, Q2 NMOS, Q3 NMOS

Commit message: adjust ICs
Parts:
- removed C7, C9: 0.1uF, Capacitor_SMD:C_0402_1005Metric, symbol Device:C
- removed U5, U6: ~, Package_SO:SSOP-24_5.3x8.2mm_P0.65mm, symbol My Parts:74LVC8T245
- added U7, U8: 74LVC541, Package_SO:TSSOP-20_4.4x6.5mm_P0.65mm, symbol 74xx:74LS541
- C2, C4, C5, C6, C8: footprint Capacitor_SMD:C_0402_1005Metric -> Capacitor_SMD:C_0603_1608Metric_Pad1.08x0.95mm_HandSolder
- Q1, Q2, Q3: value NMOS -> BSS138; footprint 0-My_Parts:MOSFET(SMD) -> Package_TO_SOT_SMD:SOT-23; symbol Simulation_SPICE:NMOS -> Transistor_FET:BSS138
- U1, U2, U3: value ~ -> (none)
- U4: value ~ -> (none); footprint Package_SO:SSOP-24_5.3x8.2mm_P0.65mm -> Package_SO:TSSOP-24_4.4x5mm_P0.4mm
Connections:
- net 3V3: now also U7.20 (VCC), U8.20 (VCC)
- net A0: now also U7.9 (A7)
- net A1: now also U7.8 (A6)
- net A2: now also U7.7 (A5)
- net A3: now also U7.6 (A4)
- net A4: now also U7.5 (A3)
- net A5: now also U7.4 (A2)
- net A6: now also U7.3 (A1)
- net A7: now also U7.2 (A0)
- net GND: now also Q1.2 (S), Q2.2 (S), Q3.2 (S), U7.10 (GND), U8.10 (GND), U8.2 (A0), U8.4 (A2), U8.6 (A4), U8.8 (A6); no longer Q1.3 (S), Q2.3 (S), Q3.3 (S)
- net SLOT_A0: now also U7.11 (Y7)
- net SLOT_A1: now also U7.12 (Y6)
- net SLOT_A2: now also U7.13 (Y5)
- net SLOT_A3: now also U7.14 (Y4)
- net SLOT_A4: now also U7.15 (Y3)
- net SLOT_A5: now also U7.16 (Y2)
- net SLOT_A6: now also U7.17 (Y1)
- net SLOT_A7: now also U7.18 (Y0)
- net SLOT_DATA_DIR: now also Q1.1 (G); no longer Q1.2 (G)
- net SLOT_INT: now also Q3.1 (G); no longer Q3.2 (G)
- net SLOT_IORQ_N: now also U8.11 (Y7)
- net SLOT_OE_N: now also U7.1 (G1), U7.19 (G2), U8.1 (G1), U8.19 (G2)
- net SLOT_RD_N: now also U8.15 (Y3)
- net SLOT_RESET_N: now also U8.17 (Y1)
- net SLOT_WAIT: now also Q2.1 (G); no longer Q2.2 (G)
- net SLOT_WR_N: now also U8.13 (Y5)
- net /BUSDIR: now also Q1.3 (D); no longer Q1.1 (D)
- net /INT: now also Q3.3 (D); no longer Q3.1 (D)
- net /IORQ: now also U8.9 (A7)
- net /RD: now also U8.5 (A3)
- net /RESET: now also U8.3 (A1)
- net /WAIT: now also Q2.3 (D); no longer Q2.1 (D)
- net /WR: now also U8.7 (A5)
Other:
- moved on the sheet: C8, J1

Commit message: *
Parts:
- removed U1: (no value), My Parts:CLOCK, symbol My Parts:CLOCK
- added X1: SG-8002DC, Package_DIP:DIP-8_W7.62mm, symbol 0_MSX:SG-8002DC
Connections:
- net 3V3: now also X1.8 (Vdd)
- net CLOCK: now also X1.5 (OUT)
- net GND: now also X1.4 (GND)
Other:
- note added: "OE は、OPEN か H で CLK を出力、L で CLK が HiZ になる。"
- note removed: "En は、OPEN か H で CLK を出力、L で CLK が HiZ になる。"
